File: fancyboard/fancyboard.kicad_pcb (KiCad board)
At the start: 2 copper layers, 48.3 x 30.5 mm, 18 parts, among them P1 USB_OTG, P2 CONN_01X08, P3 CONN_01X08, SW1 SW_Push, U1 AP111733, U2 STM32F072C8Tx

Commit message: Fixed some minor issues
Parts:
- moved C1 5.76 mm to (32.1, 31.9)
- moved G*** 1.53 mm to (31.8, 46.1)
Routing:
- net +3V3: track 112.8 -> 104.7 mm
Changed lines of the file:
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@@
-(kicad_pcb (version 4) (host pcbnew "(2016-12-22 revision d365dc590)-makepkg")
+(kicad_pcb (version 4) (host pcbnew 4.0.5)
   (general
     (links 55)
-    (no_connects 0)
+    (no_connects 1)
     (area 22.784999 22.784999 71.195001 53.415001)
     (thickness 1.6)
     (drawings 20)
-    (tracks 153)
+    (tracks 151)
     (zones 0)
     (modules 18)
@@
       (hpglpenspeed 20)
       (hpglpendiameter 15)
+      (hpglpenoverlay 2)
       (psnegative false)
       (psa4output false)
@@
   )
   (module 33c3_logo:33c3_logo (layer F.Cu)
-    (at 33.274 46.0375)
+    (at 31.75 46.101)
     (fp_text reference G*** (at 0 0) (layer F.SilkS) hide
       (effects (font (thickness 0.3)))
@@
   )
   (module Capacitors_SMD:C_0603 (layer F.Cu)
-    (at 32.766 26.15 270)
+    (at 32.131 31.877 270)
     (descr "Capacitor SMD 0603, reflow soldering, AVX (see smccp.pdf)")
     (tags "capacitor 0603")
@@
   (gr_line (start 22.86 22.86) (end 22.86 53.34) (layer Edge.Cuts) (width 0.15))
   (gr_line (start 71.12 22.86) (end 22.86 22.86) (layer Edge.Cuts) (width 0.15))
+  (segment (start 32.131 31.127) (end 32.76 31.127) (width 0.254) (layer F.Cu) (net 1))
+  (segment (start 35.439 28.448) (end 37.534315 28.448) (width 0.254) (layer F.Cu) (net 1))
+  (segment (start 32.76 31.127) (end 35.439 28.448) (width 0.254) (layer F.Cu) (net 1))
+  (segment (start 37.534315 28.448) (end 38.1 28.448) (width 0.254) (layer F.Cu) (net 1))
+  (segment (start 26.277 31.115) (end 32.119 31.115) (width 0.254) (layer F.Cu) (net 1))
+  (segment (start 32.119 31.115) (end 32.131 31.127) (width 0.254) (layer F.Cu) (net 1))
   (segment (start 58.21 33.75) (end 58.21 40.154) (width 0.254) (layer F.Cu) (net 1))
   (segment (start 58.21 40.154) (end 57.514 40.85) (width 0.254) (layer F.Cu) (net 1))
   (segment (start 57.514 40.85) (end 56.61 40.85) (width 0.254) (layer F.Cu) (net 1))
-  (segment (start 26.277 31.115) (end 32.385 31.115) (width 0.254) (layer F.Cu) (net 1))
-  (segment (start 35.052 28.448) (end 37.534315 28.448) (width 0.254) (layer F.Cu) (net 1))
-  (segment (start 32.385 31.115) (end 35.052 28.448) (width 0.254) (layer F.Cu) (net 1))
-  (segment (start 37.534315 28.448) (end 38.1 28.448) (width 0.254) (layer F.Cu) (net 1))
-  (segment (start 38.1 25.806) (end 33.172 25.806) (width 0.254) (layer F.Cu) (net 1))
-  (segment (start 33.172 25.806) (end 32.766 25.4) (width 0.254) (layer F.Cu) (net 1))
   (segment (start 50.8 50.8) (end 40.386 50.8) (width 0.254) (layer B.Cu) (net 1))
   (segment (start 40.386 50.8) (end 38.1 48.514) (width 0.254) (layer B.Cu) (net 1))
   (segment (start 38.1 48.514) (end 38.1 28.448) (width 0.254) (layer B.Cu) (net 1))
   (segment (start 38.1 32.106) (end 38.1 28.448) (width 0.254) (layer F.Cu) (net 1))
-  (segment (start 38.1 25.806) (end 38.1 27.06) (width 0.254) (layer F.Cu) (net 1))
-  (segment (start 38.1 27.06) (end 38.1 28.448) (width 0.254) (layer F.Cu) (net 1))
   (segment (start 38.1 28.584) (end 38.1 28.448) (width 0.254) (layer F.Cu) (net 1))
   (via (at 38.1 28.448) (size 0.8) (drill 0.4) (layers F.Cu B.Cu) (net 1))
