File: fancyboard/fancyboard.sch (KiCad schematic (older format))
At the start: 17 parts, among them P1 USB_OTG, P2 CONN_01X08, P3 CONN_01X08, SW1 SW_Push, U1 AP111733, U2 STM32F072C8Tx

Commit message: Fixed some minor issues
Parts:
- removed U1: AP111733, TO_SOT_Packages_SMD:SOT-223, symbol AP111733
- added U1: LM1117-3.3, symbol LM1117-3.3
Connections:
- net +3V3: now also U1.2 (VO), U1.4 (VO)
- net +5V: now also U1.3 (VI)
- net BOOT0: now also U2.44 (BOOT0)
- net GND: now also U1.1 (GND/ADJ)
- net NRST: now also U2.7 (NRST)
